File: kicad/prj/ledmat8x16tiledriver/ledmat8x16tiledriver.kicad_pcb (KiCad board)
At the start: 4 copper layers, 31.9 x 31.9 mm, 17 parts, among them J1 Conn_01x10_Pin, J2 Conn_01x10_Pin, J3 Conn_02x08_Odd_Even, J4 Conn_02x08_Odd_Even, U1 TLC59283, U2 DMP31D7LDW, U3 DMP31D7LDW, U4 DMP31D7LDW, U5 DMP31D7LDW

Commit message: Add repo url and git hash to silkscreen
For traceability, but also just becasue it's possible.
Substitution of git hash is done by kibot.
Other:
- board text added: "${git_hash}"
- board text added: "github.com/ burbschat/ledmat8x16"
Changed lines of the file:
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@@
 		(layer "Edge.Cuts")
+	)
+	(gr_text "github.com/\nburbschat/ledmat8x16"
+		(at 158.3 75.2 90)
+		(layer "B.SilkS")
+		(effects
+			(font
+				(size 1 1)
+				(thickness 0.15)
+			)
+			(justify bottom mirror)
+		)
+	)
+	(gr_text "${git_hash}"
+		(at 132.8 75.2 90)
+		(layer "B.SilkS")
+		(effects
+			(font
+				(size 1 1)
+				(thickness 0.15)
+			)
+			(justify bottom mirror)
+		)
 	)
 	(segment
